File: PCB and Schem/Devboard/HyperPlex.kicad_sch (KiCad schematic)
At the start: 33 parts, among them J1 USB_C_Receptacle_USB2.0_16P, Q1 2N3904, Q2 2N3904, Q3 2N3904, SW1 SW_Push, SW2 SW_SPDT, SW3 SW_SPDT, SW4 SW_Push, U1 CH32V203CxTx, U3 XC6206PxxxMR, U4 TP4056-42-ESOP8, U5 TPS63900, U6 XC6206PxxxMR

Commit message: Updated README, made Module 1 Schematic, started BOM
Parts:
- renumbered D2 to D1, Q3 to Q1, Q2 to Q1, R6 to R1, R4 to R1, R5 to R1, R15 to R1, R3 to R1, R7 to R10, R9 to R11, R10 to R14, R8 to R15, R13 to R3, R12 to R3, R14 to R4, R1 to R4, R11 to R9, SW4 to SW1, SW3 to SW2, U4 to U2, U5 to U2, U6 to U3
Changed lines of the file:
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@@
 		(dnp no)
 		(fields_autoplaced yes)
-		(property "Reference" "U4"
+		(property "Reference" "U2"
 			(at 263.7633 26.67 0)
 			(show_name no)
@@
 			(project "HyperPlex"
 				(path "/2159c24b-fff8-4711-9dc0-b98f0132545c"
-					(reference "U4")
+					(reference "U2")
 					(unit 1)
 				)
@@
 		(in_pos_files yes)
 		(dnp no)
-		(property "Reference" "R14"
+		(property "Reference" "R4"
 			(at 19.05 36.068 90)
 			(show_name no)
@@
 			(project "HyperPlex"
 				(path "/2159c24b-fff8-4711-9dc0-b98f0132545c"
-					(reference "R14")
+					(reference "R4")
 					(unit 1)
 				)
@@
 		(in_pos_files yes)
 		(dnp yes)
-		(property "Reference" "R9"
+		(property "Reference" "R11"
 			(at 271.78 99.822 90)
 			(show_name no)
@@
 			(project "HyperPlex"
 				(path "/2159c24b-fff8-4711-9dc0-b98f0132545c"
-					(reference "R9")
+					(reference "R11")
 					(unit 1)
 				)
@@
 		(dnp no)
 		(fields_autoplaced yes)
-		(property "Reference" "SW3"
+		(property "Reference" "SW2"
 			(at 273.05 121.9199 90)
 			(show_name no)
@@
 			(project "HyperPlex"
 				(path "/2159c24b-fff8-4711-9dc0-b98f0132545c"
-					(reference "SW3")
+					(reference "SW2")
 					(unit 1)
 				)
@@
 		(in_pos_files yes)
 		(dnp no)
-		(property "Reference" "Q3"
+		(property "Reference" "Q1"
 			(at 210.82 91.44 0)
 			(show_name no)
@@
 			(project "HyperPlex"
 				(path "/2159c24b-fff8-4711-9dc0-b98f0132545c"
-					(reference "Q3")
+					(reference "Q1")
 					(unit 1)
 				)
@@
 		(in_pos_files yes)
 		(dnp no)
-		(property "Reference" "R6"
+		(property "Reference" "R1"
 			(at 244.602 60.96 90)
 			(show_name no)
@@
 			(project "HyperPlex"
 				(path "/2159c24b-fff8-4711-9dc0-b98f0132545c"
-					(reference "R6")
+					(reference "R1")
 					(unit 1)
 				)
@@
 		(in_pos_files yes)
 		(dnp no)
-		(property "Reference" "R1"
+		(property "Reference" "R4"
 			(at 275.59 39.878 90)
 			(show_name no)
@@
 			(project "HyperPlex"
 				(path "/2159c24b-fff8-4711-9dc0-b98f0132545c"
-					(reference "R1")
+					(reference "R4")
 					(unit 1)
 				)
@@
 		(in_pos_files yes)
 		(dnp no)
-		(property "Reference" "R4"
+		(property "Reference" "R1"
 			(at 231.14 25.908 90)
 			(show_name no)
@@
 			(project "HyperPlex"
 				(path "/2159c24b-fff8-4711-9dc0-b98f0132545c"
-					(reference "R4")
+					(reference "R1")
 					(unit 1)
 				)
@@
 		(in_pos_files yes)
 		(dnp no)
-		(property "Reference" "R5"
+		(property "Reference" "R1"
 			(at 231.14 59.182 90)
 			(show_name no)
@@
 			(project "HyperPlex"
 				(path "/2159c24b-fff8-4711-9dc0-b98f0132545c"
-					(reference "R5")
+					(reference "R1")
 					(unit 1)
 				)
@@
 		(in_pos_files yes)
 		(dnp yes)
-		(property "Reference" "R7"
+		(property "Reference" "R10"
 			(at 271.78 93.218 90)
 			(show_name no)
@@
 			(project "HyperPlex"
 				(path "/2159c24b-fff8-4711-9dc0-b98f0132545c"
-					(reference "R7")
+					(reference "R10")
 					(unit 1)
 				)
@@
 		(in_pos_files yes)
 		(dnp yes)
-		(property "Reference" "R10"
+		(property "Reference" "R14"
 			(at 277.622 101.6 90)
 			(show_name no)
@@
 			(project "HyperPlex"
 				(path "/2159c24b-fff8-4711-9dc0-b98f0132545c"
-					(reference "R10")
+					(reference "R14")
 					(unit 1)
 				)
@@
 		(in_pos_files yes)
 		(dnp no)
-		(property "Reference" "D2"
+		(property "Reference" "D1"
 			(at 239.014 55.118 0)
 			(show_name no)
@@
 			(project "HyperPlex"
 				(path "/2159c24b-fff8-4711-9dc0-b98f0132545c"
-					(reference "D2")
+					(reference "D1")
 					(unit 1)
 				)
@@
 		(in_pos_files yes)
 		(dnp no)
-		(property "Reference" "R15"
+		(property "Reference" "R1"
 			(at 210.312 78.74 90)
 			(show_name no)
@@
 			(project "HyperPlex"
 				(path "/2159c24b-fff8-4711-9dc0-b98f0132545c"
-					(reference "R15")
+					(reference "R1")
 					(unit 1)
 				)
@@
 		(dnp yes)
 		(fields_autoplaced yes)
-		(property "Reference" "U5"
+		(property "Reference" "U2"
 			(at 257.81 77.47 0)
 			(show_name no)
@@
 			(project "HyperPlex"
 				(path "/2159c24b-fff8-4711-9dc0-b98f0132545c"
-					(reference "U5")
+					(reference "U2")
 					(unit 1)
 				)
@@
 		(in_pos_files yes)
 		(dnp yes)
-		(property "Reference" "R8"
+		(property "Reference" "R15"
 			(at 279.4 93.218 90)
 			(show_name no)
@@
 			(project "HyperPlex"
 				(path "/2159c24b-fff8-4711-9dc0-b98f0132545c"
-					(reference "R8")
+					(reference "R15")
 					(unit 1)
 				)
@@
 		(in_pos_files yes)
 		(dnp no)
-		(property "Reference" "R3"
+		(property "Reference" "R1"
 			(at 244.602 24.13 90)
 			(show_name no)
@@
 			(project "HyperPlex"
 				(path "/2159c24b-fff8-4711-9dc0-b98f0132545c"
-					(reference "R3")
+					(reference "R1")
 					(unit 1)
 				)
@@
 		(in_pos_files yes)
 		(dnp no)
-		(property "Reference" "Q2"
+		(property "Reference" "Q1"
 			(at 245.11 48.26 0)
 			(show_name no)
@@
 			(project "HyperPlex"
 				(path "/2159c24b-fff8-4711-9dc0-b98f0132545c"
-					(reference "Q2")
+					(reference "Q1")
 					(unit 1)
 				)
@@
 		(in_pos_files yes)
 		(dnp no)
-		(property "Reference" "#PWR02"
+		(property "Reference" "#PWR01"
 			(at 17.78 196.85 0)
 			(hide yes)
@@
 			(project "HyperPlex"
 				(path "/2159c24b-fff8-4711-9dc0-b98f0132545c"
-					(reference "#PWR02")
+					(reference "#PWR01")
 					(unit 1)
 				)
@@
 		(in_pos_files yes)
 		(dnp no)
-		(property "Reference" "R13"
+		(property "Reference" "R3"
 			(at 212.09 32.258 90)
 			(show_name no)
@@
 			(project "HyperPlex"
 				(path "/2159c24b-fff8-4711-9dc0-b98f0132545c"
-					(reference "R13")
+					(reference "R3")
 					(unit 1)
 				)
@@
 		(in_pos_files yes)
 		(dnp no)
-		(property "Reference" "SW4"
+		(property "Reference" "SW1"
 			(at 20.574 41.148 0)
 			(show_name no)
@@
 			(project "HyperPlex"
 				(path "/2159c24b-fff8-4711-9dc0-b98f0132545c"
-					(reference "SW4")
+					(reference "SW1")
 					(unit 1)
 				)
@@
 		(in_pos_files yes)
 		(dnp no)
-		(property "Reference" "U6"
+		(property "Reference" "U3"
 			(at 269.24 134.6199 90)
 			(show_name no)
@@
 			(project "HyperPlex"
 				(path "/2159c24b-fff8-4711-9dc0-b98f0132545c"
-					(reference "U6")
+					(reference "U3")
 					(unit 1)
 				)
@@
 		(in_pos_files yes)
 		(dnp no)
-		(property "Reference" "#PWR01"
+		(property "Reference" "#PWR02"
 			(at 22.86 194.31 0)
 			(hide yes)
@@
 			(project "HyperPlex"
 				(path "/2159c24b-fff8-4711-9dc0-b98f0132545c"
-					(reference "#PWR01")
+					(reference "#PWR02")
 					(unit 1)
 				)
@@
 		(in_pos_files yes)
 		(dnp no)
-		(property "Reference" "R12"
+		(property "Reference" "R3"
 			(at 212.09 38.862 90)
 			(show_name no)
@@
 			(project "HyperPlex"
 				(path "/2159c24b-fff8-4711-9dc0-b98f0132545c"
-					(reference "R12")
+					(reference "R3")
 					(unit 1)
 				)
@@
 		(in_pos_files yes)
 		(dnp yes)
-		(property "Reference" "R11"
+		(property "Reference" "R9"
 			(at 270.002 104.14 90)
 			(show_name no)
@@
 			(project "HyperPlex"
 				(path "/2159c24b-fff8-4711-9dc0-b98f0132545c"
-					(reference "R11")
-					(unit 1)
-				)
+					(reference "R9")
+					(unit 1)
+				)
